Commit message: m5 ex04 not done

File: module5/ex04/circle_movement/description/fox.urdf (robot description, URDF)
Before this commit: robot sam_bot, 16 links, 15 joints
Links:
- link left_eye_reflect: geometry collision box size=0.0025 0.04 0.04; visual box size=0.0025 0.04 0.04
- link right_eye_reflect: geometry collision box size=0.0025 0.04 0.04; visual box size=0.0025 0.04 0.04
Joints:
- joint left_eye_reflect_joint: origin xyz=0.1575 -0.1 0.095 rpy=0 0 0 -> xyz=0.15875 -0.1 0.095 rpy=0 0 0
- joint right_eye_reflect_joint: origin xyz=0.1575 0.06 0.095 rpy=0 0 0 -> xyz=0.15875 0.06 0.095 rpy=0 0 0

File: module5/ex04/circle_movement/description/fox.urdf.xacro (robot description, xacro)
@@ -1,4 +1,4 @@
 <?xml version="1.0"?>
-<robot name="sam_bot" xmlns:xacro="http://ros.org/wiki/xacro">
+<robot name="foxy" xmlns:xacro="http://ros.org/wiki/xacro">
   <xacro:include filename="gazebo.urdf.xacro" />
   <!-- Define robot constants -->
@@ -16,5 +16,5 @@
   <xacro:property name="eye_height" value="0.08"/>
   <xacro:property name="eye_reflect_width" value="0.04"/>
-  <xacro:property name="eye_reflect_length" value="0.005"/>
+  <xacro:property name="eye_reflect_length" value="0.0025"/>
   <xacro:property name="eye_reflect_height" value="0.04"/>
   <xacro:property name="cheek_width" value="0.15"/>
@@ -29,10 +29,10 @@
   <xacro:property name="wheel_radius" value="0.10"/>
   <xacro:property name="wheel_width" value="0.04"/>
-  <xacro:property name="wheel_ygap" value="0.025"/>
+  <xacro:property name="wheel_ygap" value="0.02"/>
   <xacro:property name="wheel_zoff" value="0.08"/>
   <xacro:property name="wheel_xoff" value="0.12"/>
   <xacro:property name="caster_xoff" value="0.11"/>
   <material name="Orange">
-    <color rgba="1. 0.404 0.0 1.0"/>
+    <color rgba="0.9921568627450981 0.13529411764705882 0.023529411764705882 1.0"/>
   </material>
   <material name="White">
@@ -40,5 +40,5 @@
   </material>
   <material name="Black">
-    <color rgba="0. 0. 0.0 0.0"/>
+    <ambient> 0. 0. 0.0 0.0"</ambient>
   </material>
   <!-- Define intertial property macros  -->
@@ -174,5 +174,5 @@
       <parent link="base_link"/>
       <child link="${prefix}_eye_reflect"/>
-      <origin xyz="${base_height/2+eye_reflect_length/2} ${-(0.08+0.02)+(y_reflect*(0.08+0.02+0.06))} ${-(wheel_radius+wheel_zoff-base_height/2-0.12)}" rpy="0 0 0"/>
+      <origin xyz="${base_height/2+(eye_reflect_length+eye_length)/2} ${-(0.08+0.02)+(y_reflect*(0.08+0.02+0.06))} ${-(wheel_radius+wheel_zoff-base_height/2-0.12)}" rpy="0 0 0"/>
     </joint>
   </xacro:macro>
@@ -246,7 +246,5 @@
             <cylinder radius="${wheel_radius}" length="${wheel_width}"/>
         </geometry>
-        <material name="Cyan">
-          <color rgba="0.5 0.5 0.5 1.0"/>
-        </material>
+        <material name="White"/>
       </visual>
       <collision>
@@ -265,6 +263,6 @@
     </joint>
   </xacro:macro>
-  <xacro:wheel prefix="drivewhl_l" x_reflect="-1" y_reflect="1" />
-  <xacro:wheel prefix="drivewhl_r" x_reflect="-1" y_reflect="-1" />
+  <xacro:wheel prefix="left_wheel" x_reflect="-1" y_reflect="1" />
+  <xacro:wheel prefix="right_wheel" x_reflect="-1" y_reflect="-1" />
   <!-- Caster Wheel -->
   <link name="front_caster">
@@ -273,7 +271,5 @@
         <sphere radius="${(wheel_radius+wheel_zoff-(base_height/2))}"/>
       </geometry>
-      <material name="Cyan">
-        <color rgba="0 1.0 1.0 1.0"/>
-      </material>
+      <material name="Orange"/>
     </visual>
     <collision>
@@ -285,5 +281,5 @@
     <xacro:sphere_inertia m="0.5" r="${(wheel_radius+wheel_zoff-(base_height/2))}"/>
   </link>
-  <joint name="caster_joint" type="fixed">
+  <joint name="caster_joint" type="continuous">
     <parent link="base_link"/>
     <child link="front_caster"/>

File: module5/ex04/circle_movement/description/gazebo.urdf.xacro (robot description, xacro)
@@ -24,7 +24,7 @@
             filename="gz-sim-diff-drive-system"
             name="gz::sim::systems::DiffDrive">
-            <left_joint>drivewhl_l_joint</left_joint>
-            <right_joint>drivewhl_r_joint</right_joint>
-            <child_frame_id>robot/base_link</child_frame_id>
+            <left_joint>left_wheel_joint</left_joint>
+            <right_joint>right_wheel_joint</right_joint>
+            <child_frame_id>fox/base_link</child_frame_id>
             <wheel_separation>0.35</wheel_separation>
             <wheel_radius>0.1</wheel_radius>
