Commit message: done

File: module6/ex01/circle_movement/description/fox_lidar.urdf.xacro (robot description, xacro)
@@ -42,5 +42,4 @@
   <material name="Black">
     <ambient> 0. 0. 0.0 0.0"</ambient>
-    <color rgba="0. 0. 0.0 0.0"/>
   </material>
   <!-- Define intertial property macros  -->

File: module6/ex01/circle_movement/description/lidar.urdf.xacro (robot description, xacro)
@@ -2,10 +2,10 @@
 <robot xmlns:xacro="http://www.ros.org/wiki/xacro">
     <material name="black">
-      <color rgba="0. 0. 0.0 0.0"/>
+      <ambient> 0. 0. 0.0 0.0"</ambient>
     </material>
     <joint name="laser_joint" type="fixed">
         <parent link="base_link"/>
         <child link="laser_frame"/>
-        <origin xyz="0.1 0 0.212" rpy="0 0 0"/>
+        <origin xyz="0.1 0 0.25" rpy="0 0 0"/>
     </joint>
     <link name="laser_frame">
